File: ToiletLock/ToiletLock.sch (KiCad schematic (older format))
At the start: 27 parts, among them J1 Conn_01x02_Male, U1 DRV8837C, U2 APDS-9960, Y1 Crystal_GND24

Commit message: del useless file
Parts:
- L1: footprint Inductor_SMD:L_Taiyo-Yuden_NR-50xx_HandSoldering -> Inductor_SMD:L_Bourns-SRN4018
- U2: footprint APDS-9960 -> Silicon-Custom:APDS-9960
Connections:
- net GND: now also U1.4 (GND), U1.9 (GND)
Changed lines of the file:
@@
 F 0 "L1" V 8890 1700 50  0000 C CNN
 F 1 "2.2uH 2.6A" V 8799 1700 50  0000 C CNN
-F 2 "Inductor_SMD:L_Taiyo-Yuden_NR-50xx_HandSoldering" H 8700 1700 50  0001 C CNN
+F 2 "Inductor_SMD:L_Bourns-SRN4018" H 8700 1700 50  0001 C CNN
 F 3 "~" H 8700 1700 50  0001 C CNN
 	1    8700 1700
@@
 F 0 "U2" H 6000 5510 45  0000 C CNN
 F 1 "APDS-9960" H 6000 5426 45  0000 C CNN
-F 2 "APDS-9960" H 6000 5350 20  0001 C CNN
+F 2 "Silicon-Custom:APDS-9960" H 6000 5350 20  0001 C CNN
 F 3 "" H 6000 4950 60  0001 C CNN
 F 4 "SEN-12005" H 6000 5331 60  0000 C CNN "Field4"
@@
 Text Label 1950 3050 0    50   ~ 0
 SCL
+Wire Wire Line
+	2550 5350 2700 5350
 $EndSCHEMATC
