File: Toiletlock-V2/Toiletlock-V2.kicad_pcb (KiCad board)
At the start: 2 copper layers, 12 parts, among them J1 Conn_ARM_JTAG_SWD_20, J2 Conn_ST_STDC14, SW1 SW_Push, U1 STM32G031K8T3, Y1 Crystal_GND24

Commit message: V2Sch
Parts:
- added BATT1: Conn_01x02_Male, Connector_JST:JST_PH_B2B-PH-K_1x02_P2.00mm_Vertical, F.Cu at (134.6, 120.7)
- added C4: 0.1uF, Capacitor_SMD:C_0603_1608Metric, F.Cu at (151.9, 109.5)
- added C5: 0.1uF, Capacitor_SMD:C_0603_1608Metric, F.Cu at (151.9, 112.0)
- added C6: 0.1uF, Capacitor_SMD:C_0603_1608Metric, F.Cu at (141.6, 122.3)
- added Cin1: 4.7uF, Capacitor_SMD:C_0603_1608Metric, F.Cu at (151.8, 114.9)
- added Cout1: 10uF, Capacitor_SMD:C_0603_1608Metric, F.Cu at (145.7, 120.0)
- added J2: Conn_01x02_Male, Connector_JST:JST_PH_S2B-PH-K_1x02_P2.00mm_Horizontal, F.Cu at (134.6, 110.7)
- added L1: 2.2uH 2.6A, Inductor_SMD:L_Bourns-SRN4018, F.Cu at (142.7, 111.0)
- added LED1: LED, LED_SMD:LED_0603_1608Metric, F.Cu at (141.6, 119.8)
- added ON1: LED, LED_SMD:LED_0603_1608Metric, F.Cu at (147.8, 115.0)
- added R1: 22R, Resistor_SMD:R_0603_1608Metric, F.Cu at (146.4, 117.5)
- added RLED1: 1k, Resistor_SMD:R_0603_1608Metric, F.Cu at (149.7, 120.0)
- added RON1: 1k, Resistor_SMD:R_0603_1608Metric, F.Cu at (154.5, 117.4)
- added RRX1: 22R, Resistor_SMD:R_0603_1608Metric, F.Cu at (149.6, 122.5)
- added RTX1: 22R, Resistor_SMD:R_0603_1608Metric, F.Cu at (153.7, 120.0)
- added Rfbb1: 100k, Resistor_SMD:R_0603_1608Metric, F.Cu at (150.5, 117.5)
- added Rfbt1: 453k, Resistor_SMD:R_0603_1608Metric, F.Cu at (145.6, 122.5)
- added TLV62568DBVR1: TLV62568DBV, Package_TO_SOT_SMD:SOT-23-5, F.Cu at (142.0, 116.2)
- added U2: DRV8837C, Package_SON:WSON-8-1EP_2x2mm_P0.5mm_EP0.9x1.6mm, F.Cu at (129.2, 122.3)
- added U3: APDS-9960, Silicon-Custom:APDS-9960, F.Cu at (147.5, 111.1)
- added UART1: Conn_01x04_Female, Connector_PinSocket_2.54mm:PinSocket_1x04_P2.54mm_Vertical, F.Cu at (129.4, 110.6)
- moved Y1 47.1 mm to (142.2, 100.3)
- renumbered J2 to J1, J1 to J3
Connections:
- CL1 pad 2: Net-(CL1-Pad2) -> GND
- CL2 pad 2: Net-(CL1-Pad2) -> GND
- U1 pad 20: Net-(U1-Pad20) -> /PC6

Commit message: module
Parts:
- SW1: footprint Button_Switch_THT:SW_PUSH_6mm_H5mm -> Button_Switch_SMD:SW_SPST_PTS810
- moved BATT1 44.8 mm to (177.4, 107.3)
- moved C4 44.8 mm to (194.7, 96.2)
- moved C5 44.8 mm to (194.7, 98.7)
- moved Cout1 44.8 mm to (188.4, 106.7)
- moved J2 44.8 mm to (177.4, 97.3)
- moved ON1 44.8 mm to (190.5, 101.6)
- moved RLED1 44.8 mm to (192.4, 106.7)
- moved RON1 44.8 mm to (197.2, 104.1)
- moved RTX1 44.8 mm to (196.4, 106.7)
- moved TLV62568DBVR1 44.8 mm to (184.8, 102.8)
- moved U3 44.8 mm to (190.3, 97.7)
- moved C6 44.8 mm to (184.4, 109.0)
- moved Cin1 44.8 mm to (194.5, 101.6)
- moved L1 44.8 mm to (185.4, 97.7)
- moved LED1 44.8 mm to (184.4, 106.4)
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Other:
- board outline added: 100 x 100 mm

Commit message: Dev board finish
Parts:
- moved RLED1 59.2 mm to (134.5, 94.8), turned to 180 degrees
- moved LED1 46.9 mm to (139.0, 94.8)
- moved J3 24.8 mm to (126.4, 68.0), turned to 90 degrees
- moved C6 13.8 mm to (175.2, 98.6)
- moved Cin1 12.9 mm to (185.4, 92.4)
- moved L1 12.9 mm to (176.3, 88.6)
- moved RRX1 12.9 mm to (183.3, 100.0)
- moved Rfbb1 12.9 mm to (184.1, 95.0)
- moved U3 12.9 mm to (181.1, 88.6)
- moved UART1 12.9 mm to (163.0, 88.1)
- moved BATT1 12.9 mm to (168.3, 98.2)
- moved C4 12.9 mm to (185.6, 87.1)
- moved C5 12.9 mm to (185.6, 89.6)
- moved Cout1 12.9 mm to (179.3, 97.5)
- moved J2 12.9 mm to (168.3, 88.2)
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Routing:
- net /NRST: track 0.00 -> 57.4 mm, vias 0 -> 2
- net GND: track 0.00 -> 49.8 mm, vias 0 -> 1
- net T_VCP_TX: track 0.00 -> 31.9 mm, vias 0 -> 2
- net /PB3: track 0.00 -> 26.8 mm, vias 0 -> 1
- net VDD: track 0.00 -> 24.9 mm, vias 0 -> 2
- net T_VCP_RX: track 0.00 -> 24.3 mm, vias 0 -> 2
- net /PB4: track 0.00 -> 23.7 mm, vias 0 -> 1
- net /PA8: track 0.00 -> 22.1 mm, vias 0 -> 3
- net /PB5: track 0.00 -> 20.0 mm, vias 0 -> 1
- net Net-(CL1-Pad1): track 0.00 -> 19.1 mm
- net Net-(CL2-Pad1): track 0.00 -> 18.6 mm
- net /PB6: track 0.00 -> 17.9 mm
- net /PB1: track 0.00 -> 16.8 mm, vias 0 -> 1
- net /PB7: track 0.00 -> 15.7 mm
- net /PB2: track 0.00 -> 15.3 mm, vias 0 -> 1
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- added copper zone on F.Cu, net GND
- added copper zone on B.Cu, net VDD

Commit message: arrange peripheral
Parts:
- moved C4 85.3 mm to (103.3, 64.4)
- moved C5 85.3 mm to (103.3, 67.0)
- moved RTX1 72.0 mm to (115.7, 104.8)
- moved RRX1 67.2 mm to (116.1, 101.0)
- moved J2 66.1 mm to (111.2, 54.8)
- moved U2 61.9 mm to (110.9, 66.1)
- moved RON1 58.9 mm to (136.8, 123.8)
- moved ON1 57.6 mm to (133.0, 123.8), turned to 180 degrees
- moved UART1 54.4 mm to (109.4, 97.4)
- moved Cin1 39.3 mm to (179.0, 131.2)
- moved BATT1 38.9 mm to (166.3, 137.0)
- moved Rfbt1 36.1 mm to (186.1, 135.5)
- moved Rfbb1 36.0 mm to (185.6, 130.9)
- moved L1 34.8 mm to (168.8, 122.6)
- moved TLV62568DBVR1 29.5 mm to (177.7, 123.1)
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Connections:
- A1 pad 17: VDD -> +3V3
- C1 pad 1: VDD -> +3V3
- C2 pad 1: VDD -> +3V3
- J1 pad 3: VDD -> +3V3
- J3 pad 1: VDD -> +3V3
- J3 pad 2: VDD -> +3V3
- JP1 pad 2: VDD -> +3V3
- U1 pad 4: VDD -> +3V3
Routing:
- net +3V3: track 0.00 -> 33.1 mm, vias 0 -> 2
- net VDD: track 24.9 -> 0.00 mm, vias 2 -> 0
- net GND: track 49.8 -> 54.2 mm
- net Net-(ON1-Pad1): track 0.00 -> 2.20 mm
- added copper zone on B.Cu, net +3V3
- removed copper zone on B.Cu, net VDD

Commit message: tomorrow continue
Parts:
- added C7: CP 10uF, Capacitor_SMD:C_0603_1608Metric, F.Cu at (163.5, 70.0)
- added C8: 1uF, Capacitor_SMD:C_0603_1608Metric, F.Cu at (170.4, 75.1)
- added JP10: SolderJumper_2_Open, Jumper:SolderJumper-2_P1.3mm_Open_TrianglePad1.0x1.5mm, F.Cu at (83.5, 72.5)
- added JP2: SolderJumper_2_Bridged, Jumper:SolderJumper-2_P1.3mm_Bridged_Pad1.0x1.5mm, F.Cu at (182.8, 67.5)
- added JP3: SolderJumper_2_Bridged, Jumper:SolderJumper-2_P1.3mm_Bridged_Pad1.0x1.5mm, F.Cu at (182.8, 71.3)
- added JP4: SolderJumper_2_Bridged, Jumper:SolderJumper-2_P1.3mm_Bridged_Pad1.0x1.5mm, F.Cu at (182.8, 75.1)
- added JP5: SolderJumper_2_Open, Jumper:SolderJumper-2_P1.3mm_Open_TrianglePad1.0x1.5mm, F.Cu at (182.7, 79.1)
- added JP6: SolderJumper_2_Open, Jumper:SolderJumper-2_P1.3mm_Open_TrianglePad1.0x1.5mm, F.Cu at (182.7, 82.9)
- added JP7: SolderJumper_2_Open, Jumper:SolderJumper-2_P1.3mm_Open_TrianglePad1.0x1.5mm, F.Cu at (182.6, 86.9)
- added JP8: SolderJumper_2_Open, Jumper:SolderJumper-2_P1.3mm_Open_TrianglePad1.0x1.5mm, F.Cu at (83.9, 60.9)
- added JP9: SolderJumper_2_Open, Jumper:SolderJumper-2_P1.3mm_Open_TrianglePad1.0x1.5mm, F.Cu at (83.7, 66.2)
- added RP1: 4.7k, Resistor_SMD:R_0603_1608Metric, F.Cu at (191.4, 68.5)
- added RP2: 4.7k, Resistor_SMD:R_0603_1608Metric, F.Cu at (191.4, 71.3)
- added RP3: 10k, Resistor_SMD:R_0603_1608Metric, F.Cu at (191.4, 74.1)
- added Test1: Conn_01x05, Connector_PinHeader_2.54mm:PinHeader_1x05_P2.54mm_Vertical, F.Cu at (170.9, 60.1)
- added Test2: Conn_01x06, Connector_PinHeader_2.54mm:PinHeader_1x06_P2.54mm_Vertical, F.Cu at (118.5, 64.7)
- added Test3: Conn_01x03, Connector_PinHeader_2.54mm:PinHeader_1x03_P2.54mm_Vertical, F.Cu at (188.4, 114.7)
- added Test4: Conn_01x02, Connector_PinHeader_2.54mm:PinHeader_1x02_P2.54mm_Vertical, F.Cu at (109.7, 74.8)
- C6: value 0.1uF -> 1uF
- moved C6 11.1 mm to (168.6, 70.0), turned to 270 degrees
- moved R1 9.34 mm to (167.6, 66.4), turned to 180 degrees
- moved U3 1.80 mm to (173.9, 70.5)
Connections:
- R1 pad 1: +3V3 -> Net-(C6-Pad1)
- R1 pad 2: Net-(C6-Pad1) -> +3V3
- U2 pad 5: /PB8 -> Net-(JP10-Pad2)
- U2 pad 6: /PB7 -> Net-(JP9-Pad2)
- U2 pad 7: /PB6 -> Net-(JP8-Pad2)
- U3 pad 1: /PA10 -> Net-(JP2-Pad1)
- U3 pad 2: /INT -> Net-(JP4-Pad1)
- U3 pad 3: +3V3 -> Net-(U3-Pad3)
- U3 pad 4: +3V3 -> Net-(U3-Pad3)
- U3 pad 7: /PA9 -> Net-(JP3-Pad1)
Routing:
- net Net-(JP3-Pad1): track 0.00 -> 40.4 mm, vias 0 -> 4
- net Net-(JP2-Pad1): track 0.00 -> 39.2 mm, vias 0 -> 2
- net +3V3: track 33.1 -> 72.2 mm
- net GND: track 54.2 -> 81.4 mm, vias 1 -> 2
- net Net-(JP4-Pad1): track 0.00 -> 26.9 mm, vias 0 -> 1
- net Net-(C6-Pad1): track 0.00 -> 7.57 mm
- net Net-(JP4-Pad2): track 0.00 -> 7.52 mm
- net Net-(JP2-Pad2): track 0.00 -> 7.52 mm
- net Net-(JP3-Pad2): track 0.00 -> 7.10 mm
- net /PA8: track 22.1 -> 28.1 mm
- net Net-(U3-Pad3): track 0.00 -> 0.97 mm

Commit message: Update Toiletlock-V2.kicad_pcb
Parts:
- moved JP8 42.6 mm to (118.3, 86.0), turned to 180 degrees
- moved JP9 42.4 mm to (118.3, 90.8), turned to 180 degrees
- moved UART1 42.1 mm to (135.9, 64.8)
- moved JP10 41.6 mm to (118.3, 95.4), turned to 180 degrees
- moved RTX1 41.0 mm to (140.8, 72.4)
- moved RRX1 39.9 mm to (140.8, 69.6)
- moved Test2 35.3 mm to (106.3, 97.8), turned to 180 degrees
- moved BATT1 30.6 mm to (196.5, 132.2), turned to 180 degrees
- moved Cout1 25.3 mm to (181.4, 140.2)
- moved Cin1 18.9 mm to (195.8, 140.0)
- moved C4 18.1 mm to (119.2, 73.0), turned to 180 degrees
- moved L1 13.7 mm to (178.1, 132.6), turned to 180 degrees
- moved TLV62568DBVR1 12.0 mm to (186.1, 131.7)
- moved Test4 11.8 mm to (113.3, 63.6), turned to 270 degrees
- moved Rfbt1 10.3 mm to (184.5, 125.4)
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Routing:
- net GND: track 81.4 -> 702.1 mm, vias 2 -> 6
- net +3V3: track 72.2 -> 499.5 mm, vias 2 -> 5
- net +3V8: track 0.00 -> 171.4 mm, vias 0 -> 1
- net /PA9: track 12.8 -> 139.7 mm, vias 1 -> 2
- net /PA10: track 10.8 -> 137.0 mm, vias 1 -> 2
- net /PA8: track 28.1 -> 139.9 mm, vias 3 -> 4
- net /SWCLK: track 12.9 -> 55.2 mm
- net Net-(JP10-Pad2): track 0.00 -> 40.7 mm, vias 0 -> 1
- net Net-(JP9-Pad2): track 0.00 -> 37.9 mm, vias 0 -> 1
- net Net-(J2-Pad1): track 0.00 -> 37.5 mm
- net /NRST: track 57.4 -> 93.7 mm
- net Net-(JP8-Pad2): track 0.00 -> 35.1 mm, vias 0 -> 1
- net /SWDIO: track 13.6 -> 45.2 mm
- net Net-(J2-Pad2): track 0.00 -> 27.1 mm
- net T_VCP_RX: track 24.3 -> 42.9 mm
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
Commit message: finish!
Parts:
- added C10: 0.1uF, Capacitor_SMD:C_0603_1608Metric, F.Cu at (112.5, 132.0)
- added C9: 0.1uF, Capacitor_SMD:C_0603_1608Metric, F.Cu at (104.5, 146.5)
- added D1: D_Schottky, Diode_SMD:D_SMA, F.Cu at (128.5, 138.5)
- added D2: D_Schottky, Diode_SMD:D_SMA, F.Cu at (128.5, 144.5)
- added J4: USB_B_Micro, Connector_USB:USB_Micro-B_Molex-105017-0001, F.Cu at (102.8, 138.0)
- added JP11: SolderJumper_2_Open, Jumper:SolderJumper-2_P1.3mm_Open_TrianglePad1.0x1.5mm, F.Cu at (122.0, 140.0)
- added JP12: SolderJumper_2_Open, Jumper:SolderJumper-2_P1.3mm_Open_TrianglePad1.0x1.5mm, F.Cu at (122.0, 143.5)
- added U4: CH340C, Package_SO:SOIC-16_3.9x9.9mm_P1.27mm, F.Cu at (112.5, 141.0)
Routing:
- net +3V3: track 499.5 -> 394.5 mm, vias 5 -> 4
- net T_VCP_TX: track 44.8 -> 136.4 mm, vias 2 -> 6
- net T_VCP_RX: track 42.9 -> 126.6 mm, vias 2 -> 6
- net GND: track 702.1 -> 632.5 mm, vias 6 -> 8
- net Net-(JP11-Pad1): track 0.00 -> 25.3 mm
- net Net-(JP12-Pad1): track 0.00 -> 21.7 mm
- net VBUS: track 0.00 -> 20.6 mm
- net Net-(C9-Pad2): track 0.00 -> 14.4 mm
- net Net-(J4-Pad2): track 0.00 -> 9.17 mm, vias 0 -> 2
- net Net-(J4-Pad3): track 0.00 -> 7.07 mm
- net Net-(D1-Pad1): track 0.00 -> 4.40 mm
- net Net-(D2-Pad2): track 0.00 -> 4.19 mm
